File: Eagle/BDC_MotorDrv/main.brd (EAGLE design)
At the start: 100 x 80 mm, 32 parts, among them U1 ATTINY10-TSHR

Commit message: Removed redundant power filtering
Parts:
- removed C4: (no value), rcl:C0603K
- removed D2: (no value), diode:MINIMELF
- removed D3: (no value), diode:SMBJ
- removed L1: (no value), rcl:L2012C
Connections:
- removed net N$3: D2.A, D3.C, VIN.1
- removed net N$5: C4.1, D2.C, L1.1
- net GND: no longer C4.2, D3.A
- net VCC: now also VIN.1; no longer L1.2
Changed lines of the file:
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@@
 <element name="D1" library="diode" package="MINIMELF" value="" x="58.42" y="34.29" rot="MR0"/>
 <element name="C1" library="rcl" package="C0603K" value="" x="41.91" y="43.18" rot="MR0"/>
-<element name="D2" library="diode" package="MINIMELF" value="" x="6.985" y="57.785"/>
 <element name="C2" library="rcl" package="C1206K" value="" x="3.81" y="53.975" rot="R180"/>
 <element name="C3" library="rcl" package="C0603K" value="" x="3.81" y="48.895" rot="R180"/>
 <element name="LED1" library="led" package="SML0603" value="" x="-40.64" y="29.21"/>
 <element name="R2" library="rcl" package="R0603" value="" x="-24.13" y="35.56"/>
-<element name="D3" library="diode" package="SMBJ" value="" x="6.35" y="62.23" rot="R270"/>
-<element name="C4" library="rcl" package="C0603K" value="" x="-22.86" y="39.37"/>
-<element name="L1" library="rcl" package="L2012C" value="" x="3.175" y="57.15" rot="R270"/>
 <element name="VIN" library="wirepad" package="SMD1,27-2,54" value="WIREPADSMD1,27-254" x="2.54" y="64.135" rot="R90"/>
 <element name="VGND" library="wirepad" package="SMD1,27-2,54" value="WIREPADSMD1,27-254" x="2.54" y="62.23" rot="R90"/>
@@
 <contactref element="R3" pad="2"/>
 <contactref element="R4" pad="2"/>
-<contactref element="L1" pad="2"/>
 <contactref element="LED1" pad="A"/>
 <contactref element="U1" pad="5"/>
@@
 <contactref element="R6" pad="2"/>
 <contactref element="R7" pad="2"/>
+<contactref element="VIN" pad="1"/>
 <wire x1="24.35" y1="11.62" x2="52.49" y2="24.13" width="0" layer="19" extent="1-16"/>
 <wire x1="25.16" y1="6.35" x2="24.35" y2="11.62" width="0" layer="19" extent="1-1"/>
@@
 <wire x1="5.31" y1="53.975" x2="5.1054" y2="51.435" width="0" layer="19" extent="1-1"/>
 <wire x1="6.985" y1="54.19" x2="5.31" y2="53.975" width="0" layer="19" extent="1-1"/>
-<wire x1="3.175" y1="56.15" x2="5.31" y2="53.975" width="0" layer="19" extent="1-1"/>
-<wire x1="-38.52" y1="35.56" x2="3.175" y2="56.15" width="0" layer="19" extent="1-1"/>
+<wire x1="2.54" y1="64.135" x2="5.31" y2="53.975" width="0" layer="19" extent="1-1"/>
+<wire x1="-38.52" y1="35.56" x2="4.685" y2="48.895" width="0" layer="19" extent="1-1"/>
 <wire x1="-42.33" y1="35.56" x2="-38.52" y2="35.56" width="0" layer="19" extent="1-1"/>
 <wire x1="-39.89" y1="29.21" x2="-38.52" y2="35.56" width="0" layer="19" extent="1-1"/>
@@
 <wire x1="5.08" y1="40.64" x2="27.305" y2="52.07" width="0" layer="19" extent="16-16"/>
 </signal>
-<signal name="N$3">
-<contactref element="D2" pad="A"/>
-<contactref element="D3" pad="C"/>
-<contactref element="VIN" pad="1"/>
-<wire x1="2.54" y1="64.135" x2="6.35" y2="64.26" width="0" layer="19" extent="1-1"/>
-<wire x1="8.685" y1="57.785" x2="6.35" y2="64.26" width="0" layer="19" extent="1-1"/>
-</signal>
-<signal name="N$5">
-<contactref element="D2" pad="C"/>
-<contactref element="L1" pad="1"/>
-<contactref element="C4" pad="1"/>
-<wire x1="3.175" y1="58.15" x2="5.285" y2="57.785" width="0" layer="19" extent="1-1"/>
-<wire x1="-23.735" y1="39.37" x2="3.175" y2="58.15" width="0" layer="19" extent="1-1"/>
-</signal>
 <signal name="GND">
-<contactref element="D3" pad="A"/>
-<contactref element="C4" pad="2"/>
 <contactref element="VGND" pad="1"/>
 <contactref element="R2" pad="1"/>
@@
 <wire x1="6.35" y1="67.31" x2="8.89" y2="67.31" width="0" layer="19" extent="1-16"/>
 <wire x1="2.54" y1="62.23" x2="6.35" y2="67.31" width="0" layer="19" extent="1-1"/>
-<wire x1="6.35" y1="60.19" x2="2.54" y2="62.23" width="0" layer="19" extent="1-1"/>
-<wire x1="-21.985" y1="39.37" x2="2.54" y2="62.23" width="0" layer="19" extent="1-1"/>
-<wire x1="-24.98" y1="35.56" x2="-21.985" y2="39.37" width="0" layer="19" extent="1-1"/>
-<wire x1="2.31" y1="53.975" x2="6.35" y2="60.19" width="0" layer="19" extent="1-1"/>
+<wire x1="2.31" y1="53.975" x2="2.54" y2="62.23" width="0" layer="19" extent="1-1"/>
 <wire x1="2.5146" y1="51.435" x2="2.31" y2="53.975" width="0" layer="19" extent="1-1"/>
 <wire x1="2.935" y1="48.895" x2="2.5146" y2="51.435" width="0" layer="19" extent="1-1"/>
+<wire x1="-24.98" y1="35.56" x2="2.935" y2="48.895" width="0" layer="19" extent="1-1"/>
 <wire x1="26.45" y1="9.97" x2="2.935" y2="48.895" width="0" layer="19" extent="1-1"/>
 <wire x1="26.91" y1="6.35" x2="26.45" y2="9.97" width="0" layer="19" extent="1-1"/>

Commit message: Removed redundant feedback optocoupler
Parts:
- removed OK1: LTV816GEN, optocoupler:REFLECTIVE_SENSOR
- removed R6, R7: (no value), rcl:R0603
Connections:
- removed net N$2: OK1.3, R6.1
- net CLK/FEEDBACK: no longer OK1.1, R7.1
- net GND: no longer OK1.2, OK1.4
- net VCC: no longer R6.2, R7.2
Changed lines of the file:
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@@
 <attribute name="OC_FARNELL" value="unknown" x="34.925" y="13.335" size="1.778" layer="28" rot="MR0" display="off"/>
 </element>
-<element name="OK1" library="optocoupler" package="REFLECTIVE_SENSOR" value="LTV816GEN" x="7.62" y="67.31" rot="R270"/>
-<element name="R6" library="rcl" package="R0603" value="" x="-39.37" y="35.56"/>
-<element name="R7" library="rcl" package="R0603" value="" x="-43.18" y="35.56"/>
 <element name="PAD6" library="wirepad" package="SMD1,27-2,54" value="WIREPADSMD1,27-254" x="-31.75" y="25.4"/>
 <element name="PAD7" library="wirepad" package="SMD1,27-2,54" value="WIREPADSMD1,27-254" x="-35.56" y="25.4"/>
@@
 <contactref element="C5" pad="1"/>
 <contactref element="U$2" pad="4"/>
-<contactref element="R6" pad="2"/>
-<contactref element="R7" pad="2"/>
 <contactref element="VIN" pad="1"/>
 <wire x1="24.35" y1="11.62" x2="52.49" y2="24.13" width="0" layer="19" extent="1-16"/>
@@
 <wire x1="6.985" y1="54.19" x2="5.31" y2="53.975" width="0" layer="19" extent="1-1"/>
 <wire x1="2.54" y1="64.135" x2="5.31" y2="53.975" width="0" layer="19" extent="1-1"/>
-<wire x1="-38.52" y1="35.56" x2="4.685" y2="48.895" width="0" layer="19" extent="1-1"/>
-<wire x1="-42.33" y1="35.56" x2="-38.52" y2="35.56" width="0" layer="19" extent="1-1"/>
-<wire x1="-39.89" y1="29.21" x2="-38.52" y2="35.56" width="0" layer="19" extent="1-1"/>
+<wire x1="-39.89" y1="29.21" x2="4.685" y2="48.895" width="0" layer="19" extent="1-1"/>
 </signal>
 <signal name="N$1">
@@
 <contactref element="U$2" pad="2"/>
 <contactref element="C5" pad="2"/>
-<contactref element="OK1" pad="4"/>
-<contactref element="OK1" pad="2"/>
-<wire x1="6.35" y1="67.31" x2="8.89" y2="67.31" width="0" layer="19" extent="1-16"/>
-<wire x1="2.54" y1="62.23" x2="6.35" y2="67.31" width="0" layer="19" extent="1-1"/>
 <wire x1="2.31" y1="53.975" x2="2.54" y2="62.23" width="0" layer="19" extent="1-1"/>
 <wire x1="2.5146" y1="51.435" x2="2.31" y2="53.975" width="0" layer="19" extent="1-1"/>
@@
 <contactref element="U1" pad="3"/>
 <contactref element="U$2" pad="3"/>
-<contactref element="R7" pad="1"/>
-<contactref element="OK1" pad="1"/>
 <contactref element="PAD8" pad="1"/>
-<wire x1="2.5146" y1="50.4952" x2="8.89" y2="67.31" width="0" layer="19" extent="1-1"/>
 <wire x1="26.45" y1="11.62" x2="2.5146" y2="50.4952" width="0" layer="19" extent="1-1"/>
 <wire x1="-39.37" y1="25.4" x2="2.5146" y2="50.4952" width="0" layer="19" extent="1-1"/>
-<wire x1="-44.03" y1="35.56" x2="-39.37" y2="25.4" width="0" layer="19" extent="1-1"/>
-</signal>
-<signal name="N$2">
-<contactref element="OK1" pad="3"/>
-<contactref element="R6" pad="1"/>
-<wire x1="-40.22" y1="35.56" x2="6.35" y2="67.31" width="0" layer="19" extent="1-16"/>
 </signal>
 </signals>
